Commit message: Add Livox ROS Driver2 and configuration parsing for MID360 Lidar
- Implemented livox_ros_driver2.cpp for handling Lidar data publishing in ROS1 and ROS2.
- Added parse_cfg_file module for reading Lidar configuration files, including summary info and user-defined configurations.
- Created parse_livox_lidar_cfg module to handle specific Lidar configuration parsing.
- Developed tests for extrinsics and ROS types to ensure proper functionality.
- Introduced scripts for checking sensor levels and validating configurations.
- Updated soma.yaml to reflect changes in robot base frame from base_link to base_footprint.

File: examples/robot-unitree-g1/g1_description/g1_29dof.urdf (robot description, URDF)
Before this commit: robot g1_29dof, 41 links, 40 joints
Links:
- added link base_footprint
- added link livox_frame
- added link mid360_imu
- added link mid360_upright
- link head_link: geometry collision mesh filename=file:///home/szh/robonix/examples/robot-unitree-g1/g1_descr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; visual mesh filename=file:///home/szh/robonix/examples/robot-unitree-g1/g1_descr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
- link left_ankle_pitch_link: geometry collision mesh filename=file:///home/szh/robonix/examples/robot-unitree-g1/g1_descr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; visual mesh filename=file:///home/szh/robonix/examples/robot-unitree-g1/g1_descr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
- link left_ankle_roll_link: geometry collision sphere radius=0.005; collision sphere radius=0.005
- link left_elbow_link: geometry collision mesh filename=file:///home/szh/robonix/examples/robot-unitree-g1/g1_descr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; visual mesh filename=file:///home/szh/robonix/examples/robot-unitree-g1/g1_descr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
- link left_hip_pitch_link: geometry collision mesh filename=file:///home/szh/robonix/examples/robot-unitree-g1/g1_descr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; visual mesh filename=file:///home/szh/robonix/examples/robot-unitree-g1/g1_descr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
- link left_hip_roll_link: geometry collision mesh filename=file:///home/szh/robonix/examples/robot-unitree-g1/g1_descr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; visual mesh filename=file:///home/szh/robonix/examples/robot-unitree-g1/g1_descr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
- link left_hip_yaw_link: geometry collision mesh filename=file:///home/szh/robonix/examples/robot-unitree-g1/g1_descr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; visual mesh filename=file:///home/szh/robonix/examples/robot-unitree-g1/g1_descr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
- link left_knee_link: geometry collision mesh filename=file:///home/szh/robonix/examples/robot-unitree-g1/g1_descr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; visual mesh filename=file:///home/szh/robonix/examples/robot-unitree-g1/g1_descr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
- link left_rubber_hand: geometry visual mesh filename=file:///home/szh/robonix/examples/robot-unitree-g1/g1_descr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
- link left_shoulder_pitch_link: geometry collision cylinder length=0.05 radius=0.03; visual mesh filename=file:///home/szh/robonix/examples/robot-unitree-g1/g1_descr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
- link left_shoulder_roll_link: geometry collision cylinder length=0.03 radius=0.03; visual mesh filename=file:///home/szh/robonix/examples/robot-unitree-g1/g1_descr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
- link left_shoulder_yaw_link: geometry collision mesh filename=file:///home/szh/robonix/examples/robot-unitree-g1/g1_descr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; visual mesh filename=file:///home/szh/robonix/examples/robot-unitree-g1/g1_descr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
- link left_wrist_pitch_link: geometry collision mesh filename=file:///home/szh/robonix/examples/robot-unitree-g1/g1_descr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; visual mesh filename=file:///home/szh/robonix/examples/robot-unitree-g1/g1_descr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
- link left_wrist_roll_link: geometry collision mesh filename=file:///home/szh/robonix/examples/robot-unitree-g1/g1_descr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; visual mesh filename=file:///home/szh/robonix/examples/robot-unitree-g1/g1_descr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
- link left_wrist_yaw_link: geometry collision mesh filename=file:///home/szh/robonix/examples/robot-unitree-g1/g1_descr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; visual mesh filename=file:///home/szh/robonix/examples/robot-unitree-g1/g1_descr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
- link logo_link: geometry collision mesh filename=file:///home/szh/robonix/examples/robot-unitree-g1/g1_descr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; visual mesh filename=file:///home/szh/robonix/examples/robot-unitree-g1/g1_descr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
- link pelvis: geometry visual mesh filename=file:///home/szh/robonix/examples/robot-unitree-g1/g1_descr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
- link pelvis_contour_link: geometry collision mesh filename=file:///home/szh/robonix/examples/robot-unitree-g1/g1_descr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; visual mesh filename=file:///home/szh/robonix/examples/robot-unitree-g1/g1_descr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
- link right_ankle_pitch_link: geometry collision mesh filename=file:///home/szh/robonix/examples/robot-unitree-g1/g1_descr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; visual mesh filename=file:///home/szh/robonix/examples/robot-unitree-g1/g1_descr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
- link right_ankle_roll_link: geometry collision sphere radius=0.005; collision sphere radius=0.005
- link right_elbow_link: geometry collision mesh filename=file:///home/szh/robonix/examples/robot-unitree-g1/g1_descr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; visual mesh filename=file:///home/szh/robonix/examples/robot-unitree-g1/g1_descr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
- link right_hip_pitch_link: geometry collision mesh filename=file:///home/szh/robonix/examples/robot-unitree-g1/g1_descr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; visual mesh filename=file:///home/szh/robonix/examples/robot-unitree-g1/g1_descr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
- link right_hip_roll_link: geometry collision mesh filename=file:///home/szh/robonix/examples/robot-unitree-g1/g1_descr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; visual mesh filename=file:///home/szh/robonix/examples/robot-unitree-g1/g1_descr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
- link right_hip_yaw_link: geometry collision mesh filename=file:///home/szh/robonix/examples/robot-unitree-g1/g1_descr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; visual mesh filename=file:///home/szh/robonix/examples/robot-unitree-g1/g1_descr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
- link right_knee_link: geometry collision mesh filename=file:///home/szh/robonix/examples/robot-unitree-g1/g1_descr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; visual mesh filename=file:///home/szh/robonix/examples/robot-unitree-g1/g1_descr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
- link right_rubber_hand: geometry visual mesh filename=file:///home/szh/robonix/examples/robot-unitree-g1/g1_descr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
- link right_shoulder_pitch_link: geometry collision cylinder length=0.05 radius=0.03; visual mesh filename=file:///home/szh/robonix/examples/robot-unitree-g1/g1_descr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
- link right_shoulder_roll_link: geometry collision cylinder length=0.03 radius=0.03; visual mesh filename=file:///home/szh/robonix/examples/robot-unitree-g1/g1_descr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
- link right_shoulder_yaw_link: geometry collision mesh filename=file:///home/szh/robonix/examples/robot-unitree-g1/g1_descr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; visual mesh filename=file:///home/szh/robonix/examples/robot-unitree-g1/g1_descr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
- link right_wrist_pitch_link: geometry collision mesh filename=file:///home/szh/robonix/examples/robot-unitree-g1/g1_descr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; visual mesh filename=file:///home/szh/robonix/examples/robot-unitree-g1/g1_descr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
- link right_wrist_roll_link: geometry collision mesh filename=file:///home/szh/robonix/examples/robot-unitree-g1/g1_descr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; visual mesh filename=file:///home/szh/robonix/examples/robot-unitree-g1/g1_descr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
- link right_wrist_yaw_link: geometry collision mesh filename=file:///home/szh/robonix/examples/robot-unitree-g1/g1_descr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; visual mesh filename=file:///home/szh/robonix/examples/robot-unitree-g1/g1_descr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
- link torso_link: geometry collision mesh filename=file:///home/szh/robonix/examples/robot-unitree-g1/g1_descr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; visual mesh filename=file:///home/szh/robonix/examples/robot-unitree-g1/g1_descr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
- link waist_roll_link: geometry visual mesh filename=file:///home/szh/robonix/examples/robot-unitree-g1/g1_descr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
- link waist_support_link: geometry collision mesh filename=file:///home/szh/robonix/examples/robot-unitree-g1/g1_descr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; visual mesh filename=file:///home/szh/robonix/examples/robot-unitree-g1/g1_descr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
- link waist_yaw_link: geometry visual mesh filename=file:///home/szh/robonix/examples/robot-unitree-g1/g1_descr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
Joints:
- added joint base_footprint_to_base_link: type fixed, parent base_footprint, child base_link, origin xyz=0 0 0.80 rpy=0 0 0
- added joint mid360_imu_frame_joint: type fixed, parent mid360_imu, child livox_frame, origin xyz=0 0 0 rpy=3.141592653589793 0 0
- added joint mid360_imu_joint: type fixed, parent mid360_link, child mid360_imu, origin xyz=0.011 0.02329 -0.04412 rpy=0 0 0
- added joint mid360_upright_joint: type fixed, parent mid360_link, child mid360_upright, origin xyz=0 0 0 rpy=3.141592653589793 0 0
- joint mid360_joint: origin xyz=0.0002835 0.00003 0.40618 rpy=0 0.04014257279586953 0 -> xyz=0 0 0.47618 rpy=3.139111853589793 0.66736485 0; parent torso_link -> base_link

Commit message: feat: update scene-base requirements and add RealSense camera support
- Updated `scene-base.txt` to restrict `mcp` version to <2 for compatibility.
- Added a new RViz configuration file `g1.rviz` for visualizing the Unitree G1 robot.
- Introduced a new RealSense camera primitive in `main.py` with lifecycle management and image processing capabilities.
- Added unit tests for extrinsics retry logic in `test_extrinsics_retry.py`.
- Created a backup of the `robonix_manifest.yaml` for reference.
- Added a script `launch_rviz2.sh` to launch RViz with the new configuration.
- Backed up the existing `requirements.txt` for future reference.

File: examples/robot-unitree-g1/g1_description/g1_29dof.urdf (robot description, URDF)
Before this commit: robot g1_29dof, 45 links, 44 joints
Links:
- link head_link: geometry collision mesh filename=file:///data/robonix/examples/robot-unitree-g1/g1_descripti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; visual mesh filename=file:///data/robonix/examples/robot-unitree-g1/g1_descripti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
- link left_ankle_pitch_link: geometry collision mesh filename=file:///data/robonix/examples/robot-unitree-g1/g1_descripti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; visual mesh filename=file:///data/robonix/examples/robot-unitree-g1/g1_descripti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
- link left_ankle_roll_link: geometry collision sphere radius=0.005; collision sphere radius=0.005
- link left_elbow_link: geometry collision mesh filename=file:///data/robonix/examples/robot-unitree-g1/g1_descripti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; visual mesh filename=file:///data/robonix/examples/robot-unitree-g1/g1_descripti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
- link left_hip_pitch_link: geometry collision mesh filename=file:///data/robonix/examples/robot-unitree-g1/g1_descripti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; visual mesh filename=file:///data/robonix/examples/robot-unitree-g1/g1_descripti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
- link left_hip_roll_link: geometry collision mesh filename=file:///data/robonix/examples/robot-unitree-g1/g1_descripti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; visual mesh filename=file:///data/robonix/examples/robot-unitree-g1/g1_descripti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
- link left_hip_yaw_link: geometry collision mesh filename=file:///data/robonix/examples/robot-unitree-g1/g1_descripti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; visual mesh filename=file:///data/robonix/examples/robot-unitree-g1/g1_descripti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
- link left_knee_link: geometry collision mesh filename=file:///data/robonix/examples/robot-unitree-g1/g1_descripti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; visual mesh filename=file:///data/robonix/examples/robot-unitree-g1/g1_descripti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
- link left_rubber_hand: geometry visual mesh filename=file:///data/robonix/examples/robot-unitree-g1/g1_descripti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
- link left_shoulder_pitch_link: geometry collision cylinder length=0.05 radius=0.03; visual mesh filename=file:///data/robonix/examples/robot-unitree-g1/g1_descripti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
- link left_shoulder_roll_link: geometry collision cylinder length=0.03 radius=0.03; visual mesh filename=file:///data/robonix/examples/robot-unitree-g1/g1_descripti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
- link left_shoulder_yaw_link: geometry collision mesh filename=file:///data/robonix/examples/robot-unitree-g1/g1_descripti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; visual mesh filename=file:///data/robonix/examples/robot-unitree-g1/g1_descripti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
- link left_wrist_pitch_link: geometry collision mesh filename=file:///data/robonix/examples/robot-unitree-g1/g1_descripti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; visual mesh filename=file:///data/robonix/examples/robot-unitree-g1/g1_descripti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
- link left_wrist_roll_link: geometry collision mesh filename=file:///data/robonix/examples/robot-unitree-g1/g1_descripti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; visual mesh filename=file:///data/robonix/examples/robot-unitree-g1/g1_descripti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
- link left_wrist_yaw_link: geometry collision mesh filename=file:///data/robonix/examples/robot-unitree-g1/g1_descripti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; visual mesh filename=file:///data/robonix/examples/robot-unitree-g1/g1_descripti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
- link logo_link: geometry collision mesh filename=file:///data/robonix/examples/robot-unitree-g1/g1_descripti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; visual mesh filename=file:///data/robonix/examples/robot-unitree-g1/g1_descripti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
- link pelvis: geometry visual mesh filename=file:///data/robonix/examples/robot-unitree-g1/g1_descripti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
- link pelvis_contour_link: geometry collision mesh filename=file:///data/robonix/examples/robot-unitree-g1/g1_descripti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; visual mesh filename=file:///data/robonix/examples/robot-unitree-g1/g1_descripti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
- link right_ankle_pitch_link: geometry collision mesh filename=file:///data/robonix/examples/robot-unitree-g1/g1_descripti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; visual mesh filename=file:///data/robonix/examples/robot-unitree-g1/g1_descripti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
- link right_ankle_roll_link: geometry collision sphere radius=0.005; collision sphere radius=0.005
- link right_elbow_link: geometry collision mesh filename=file:///data/robonix/examples/robot-unitree-g1/g1_descripti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; visual mesh filename=file:///data/robonix/examples/robot-unitree-g1/g1_descripti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
- link right_hip_pitch_link: geometry collision mesh filename=file:///data/robonix/examples/robot-unitree-g1/g1_descripti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; visual mesh filename=file:///data/robonix/examples/robot-unitree-g1/g1_descripti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
- link right_hip_roll_link: geometry collision mesh filename=file:///data/robonix/examples/robot-unitree-g1/g1_descripti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; visual mesh filename=file:///data/robonix/examples/robot-unitree-g1/g1_descripti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
- link right_hip_yaw_link: geometry collision mesh filename=file:///data/robonix/examples/robot-unitree-g1/g1_descripti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; visual mesh filename=file:///data/robonix/examples/robot-unitree-g1/g1_descripti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
- link right_knee_link: geometry collision mesh filename=file:///data/robonix/examples/robot-unitree-g1/g1_descripti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; visual mesh filename=file:///data/robonix/examples/robot-unitree-g1/g1_descripti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
- link right_rubber_hand: geometry visual mesh filename=file:///data/robonix/examples/robot-unitree-g1/g1_descripti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
- link right_shoulder_pitch_link: geometry collision cylinder length=0.05 radius=0.03; visual mesh filename=file:///data/robonix/examples/robot-unitree-g1/g1_descripti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
- link right_shoulder_roll_link: geometry collision cylinder length=0.03 radius=0.03; visual mesh filename=file:///data/robonix/examples/robot-unitree-g1/g1_descripti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
- link right_shoulder_yaw_link: geometry collision mesh filename=file:///data/robonix/examples/robot-unitree-g1/g1_descripti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; visual mesh filename=file:///data/robonix/examples/robot-unitree-g1/g1_descripti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
- link right_wrist_pitch_link: geometry collision mesh filename=file:///data/robonix/examples/robot-unitree-g1/g1_descripti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; visual mesh filename=file:///data/robonix/examples/robot-unitree-g1/g1_descripti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
- link right_wrist_roll_link: geometry collision mesh filename=file:///data/robonix/examples/robot-unitree-g1/g1_descripti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; visual mesh filename=file:///data/robonix/examples/robot-unitree-g1/g1_descripti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
- link right_wrist_yaw_link: geometry collision mesh filename=file:///data/robonix/examples/robot-unitree-g1/g1_descripti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; visual mesh filename=file:///data/robonix/examples/robot-unitree-g1/g1_descripti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
- link torso_link: geometry collision mesh filename=file:///data/robonix/examples/robot-unitree-g1/g1_descripti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; visual mesh filename=file:///data/robonix/examples/robot-unitree-g1/g1_descripti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
- link waist_roll_link: geometry visual mesh filename=file:///data/robonix/examples/robot-unitree-g1/g1_descripti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
- link waist_support_link: geometry collision mesh filename=file:///data/robonix/examples/robot-unitree-g1/g1_descripti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; visual mesh filename=file:///data/robonix/examples/robot-unitree-g1/g1_descripti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
- link waist_yaw_link: geometry visual mesh filename=file:///data/robonix/examples/robot-unitree-g1/g1_descripti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
Joints:
- joint mid360_joint: origin xyz=0 0 0.47618 rpy=3.139111853589793 0.66736485 0 -> xyz=0 0 0.47618 rpy=3.139111853589793 0 0
